Commit message: Added rough inertial and collision model to urdf, reordered links, added dynamics (to spawn in gazebo) Fixed low-high limits order

File: flir_ptu_description/urdf/d46.urdf.xacro (robot description, xacro)
@@ -8,11 +8,12 @@
   <xacro:property name="tilt_down_range" value="0.82" />
   <xacro:property name="joint_effort" value="30" />
+  <xacro:property name="dynamic_damping" value="1.0" />
   <xacro:macro name="d46_stepper_module"
                params="ptu_name joint_name">
     <link name="${ptu_name}_${joint_name}_link">
-      <!-- <inertial>
+      <inertial>
         <mass value="0.65" />
-        <inertia ... ? />
-      </inertial> -->
+        <inertia  ixx="0.00054" ixy="0.0"  ixz="0.0"  iyy="0.00033"  iyz="0.0"	izz="0.00067" />
+      </inertial>
       <visual>
         <material name="ptu_body_color">
@@ -36,12 +37,65 @@
         <origin xyz="-0.074 0.021 0" rpy="0 1.57 0" />
       </visual>
+      <collision>
+        <geometry>
+          <box size="0.045 0.065 0.044" />
+        </geometry>
+        <origin xyz="0 0.011 0" />
+      </collision>
+      <collision>
+        <geometry>
+          <box size="0.046 0.044 0.044" />
+        </geometry>
+        <origin xyz="-0.045 0.0215 0" />
+      </collision>
     </link>
   </xacro:macro>
   <xacro:macro name="ptu_d46" params="name">
+    <link name="${name}_base_link" />
     <d46_stepper_module ptu_name="${name}" joint_name="pan" />
+    <link name="${name}_tilted_link" />
     <d46_stepper_module ptu_name="${name}" joint_name="tilt" />
-    <link name="${name}_base_link" />
-    <link name="${name}_tilted_link" />
-    <link name="${name}_mount_link" />
+    <link name="${name}_mount_link" >
+      <inertial>
+        <mass value="0.10" />
+        <inertia  ixx="0.00003" ixy="0.0"  ixz="0.0"  iyy="0.00001"  iyz="0.0"	izz="0.00004" />
+      </inertial>
+      <visual>
+        <geometry>
+          <box size="0.025 0.064 0.005" />
+        </geometry>
+        <origin xyz="0.0 0.0 -0.0025" />
+      </visual>
+      <visual>
+        <geometry>
+          <box size="0.025 0.009 0.045" />
+        </geometry>
+       <origin xyz="0.0 0.0275 -0.0275" />
+      </visual>
+      <visual>
+        <geometry>
+          <box size="0.025 0.009 0.045" />
+        </geometry>
+         <origin xyz="0.0 -0.0275 -0.0275" />
+      </visual>
+      <collision>
+        <geometry>
+          <box size="0.025 0.064 0.005" />
+        </geometry>
+        <origin xyz="0.0 0.0 -0.0025" />
+      </collision>
+      <collision>
+        <geometry>
+          <box size="0.025 0.009 0.045" />
+        </geometry>
+        <origin xyz="0.0 0.0275 -0.0275" />
+      </collision>
+      <collision>
+        <geometry>
+          <box size="0.025 0.009 0.045" />
+        </geometry>
+        <origin xyz="0.0 -0.0275 -0.0275" />
+      </collision>
+    </link>
     <!-- There's an offset between the origin of the pan joint and the origin of
          the overall device, which is between the mounting screws on its base. -->
@@ -57,6 +111,7 @@
       <child link="${name}_tilt_link" />
       <axis xyz="0 1 0" rpy="0 0 0" />
-      <limit lower="${pan_range}" upper="${-pan_range}"
+      <limit lower="${-pan_range}" upper="${pan_range}"
              effort="${joint_effort}" velocity="${pan_velocity}" />
+      <dynamics friction="10.0" damping="${dynamic_damping}"/>
     </joint>
     <!-- The tilt joint -->
@@ -68,4 +123,5 @@
       <limit lower="${-tilt_down_range}" upper="${tilt_up_range}"
              effort="${joint_effort}" velocity="${tilt_velocity}" />
+      <dynamics friction="10.0" damping="${dynamic_damping}"/>
     </joint>
     <!-- Fixed joint to provide a convenient attachment point for accessories. -->

Commit message: Fixed sign in description to match real device

File: flir_ptu_description/urdf/d46.urdf.xacro (robot description, xacro)
@@ -110,5 +110,5 @@
       <origin xyz="0 0 0.066" rpy="-1.5708 0 0" />
       <child link="${name}_tilt_link" />
-      <axis xyz="0 1 0" rpy="0 0 0" />
+      <axis xyz="0 -1 0" rpy="0 0 0" />
       <limit lower="${-pan_range}" upper="${pan_range}"
              effort="${joint_effort}" velocity="${pan_velocity}" />
